File: pcb/astrotracker.kicad_sch (KiCad schematic)
At the start: 0 parts

Commit message: pcb design
Parts:
- added M1, M2, M3: Stepper_Motor_bipolar, symbol Motor:Stepper_Motor_bipolar
- added NEO-8M1: ~, NEO-8M:GPS NEO-8M, symbol NEO_8M-symbol:GPS_NEO-8M
- added QMC5883L_COMPASS1: ~, symbol QMC5883L:QMC5883L
- added R1, R2, R3, R4, R5, R6, R7: 10K, symbol Device:R
- added SW1, SW2, SW3, SW4, SW5, SW6, SW7: SW_Push_Open_Dual, symbol Switch:SW_Push_Open_Dual
- added U1: DEVKIT_V1_ESP32-WROOM-32, DEVKIT_V1_ESP32-WROOM-32:MODULE_DEVKIT_V1_ESP32-WROOM-32, symbol DEVKIT_V1_ESP32-WROOM-32:DEVKIT_V1_ESP32-WROOM-32
- added U2, U3, U4: TMC2209_SILENTSTEPSTICK, TMC2209_SILENTSTEPSTICK:MODULE_TMC2209_SILENTSTEPSTICK, symbol TMC2209_MODULE:TMC2209_SILENTSTEPSTICK
- added i2c_LCD1: ~, symbol i2c_LCD:i2c_LCD
Connections:
- new net: NEO-8M1. (GND), QMC5883L_COMPASS1. (VCC), SW1.1, SW2.1, SW3.1, SW4.1, SW5.1, SW6.1, SW7.1, U1.1 (3V3), U2.2 (VIO), U3.2 (VIO), U4.2 (VIO), i2c_LCD1. (SCL)
- new net: R1.1, SW7.3
- new net: SW7.4, U1.11 (IO27)
- new net: QMC5883L_COMPASS1. (VCC), U1.33 (IO21), i2c_LCD1. (SCL)
- new net: QMC5883L_COMPASS1. (VCC), U1.36 (IO22), i2c_LCD1. (SCL)
- new net: QMC5883L_COMPASS1. (VCC), U1.38 (GND3), i2c_LCD1. (SCL)
- new net: R4.1, SW2.3
- new net: R1.2, R2.2, R3.2, R4.2, R5.2, R6.2, R7.2, U1.14 (GND1)
- new net: U1.26 (IO4), U2.10 (STEP)
- new net: U1.28 (IO17), U2.11 (PDN), U2.12 (UART), U3.11 (PDN), U3.12 (UART), U4.11 (PDN), U4.12 (UART)
- new net: U1.31 (IO19), U2.16 (~{EN})
- new net: M1.3, U2.3 (M1B)
- new net: M1.1, U2.4 (M1A)
- new net: M1.2 (-), U2.5 (M2A)
- new net: M1.4, U2.6 (M2B)
- new net: U1.23 (IO15), U2.9 (DIR)
- new net: R5.1, SW5.3
- new net: SW5.4, U1.9 (IO25)
- new net: U1.24 (IO2), U4.10 (STEP)
- new net: U1.29 (IO5), U4.16 (~{EN})
- new net: M3.3, U4.3 (M1B)
- new net: M3.1, U4.4 (M1A)
- new net: M3.2 (-), U4.5 (M2A)
- new net: M3.4, U4.6 (M2B)
- new net: U1.21 (SD0), U4.9 (DIR)
- new net: R7.1, SW3.3
- new net: SW3.4, U1.7 (IO32)
- new net: M2.1, U3.4 (M1A)
- new net: M2.2 (-), U3.5 (M2A)
- new net: M2.3, U3.3 (M1B)
- new net: M2.4, U3.6 (M2B)
- new net: R2.1, SW4.3
- new net: SW4.4, U1.8 (IO33)
- new net: NEO-8M1. (GND), U1.32 (GND2)
- new net: NEO-8M1. (GND), U1.34 (RXD0)
- new net: NEO-8M1. (GND), U1.35 (TXD0)
- new net: SW2.4, U1.6 (IO35)
- new net: U1.25 (IO0), U3.10 (STEP)
- new net: U1.30 (IO18), U3.16 (~{EN})
- new net: U1.22 (SD1), U3.9 (DIR)
- new net: SW6.4, U1.10 (IO26)
- new net: SW1.4, U1.5 (IO34)
- new net: R3.1, SW1.3
- new net: R6.1, SW6.3
- new net +22.2V-25.2V (6S LiPo): U2.8 (VM), U3.8 (VM), U4.8 (VM)
- new net GND (6S LiPo): U2.1 (GND), U2.7 (GND), U3.1 (GND), U3.7 (GND), U4.1 (GND), U4.7 (GND)
Other:
- note added: "Astrotracker H1"
- note added: "June 25, 2025"
- note added: "v1.0"

Commit message: finish pcb
Parts:
- removed NEO-8M1: ~, NEO-8M:GPS NEO-8M, symbol NEO_8M-symbol:GPS_NEO-8M
- removed QMC5883L_COMPASS1: ~, symbol QMC5883L:QMC5883L
- removed i2c_LCD1: ~, symbol i2c_LCD:i2c_LCD
- added U5: QMC5883L_COMPASS, QMC5883L:QMC5883L, symbol QMC5883L:QMC5883L
- added U6: NEO-8M, NEO-8M:GPS NEO-8M, symbol NEO_8M-symbol:GPS_NEO-8M
- added U7: i2c_LCD, i2c_LCD:i2c_LCD, symbol i2c_LCD:i2c_LCD
- M1, M2, M3: footprint (none) -> NEMA_17:NEMA-17
- R1, R2, R3, R4, R5, R6, R7: footprint (none) -> Resistor_THT:R_Axial_DIN0207_L6.3mm_D2.5mm_P7.62mm_Horizontal
- SW1, SW2, SW3, SW4, SW5, SW6, SW7: value SW_Push_Open_Dual -> SW_Push; footprint (none) -> Button_Switch_THT:SW_PUSH_6mm; symbol Switch:SW_Push_Open_Dual -> Switch:SW_Push
- U2, U3, U4: footprint TMC2209_SILENTSTEPSTICK:MODULE_TMC2209_SILENTSTEPSTICK -> TMC2209_MODULE:MODULE_TMC2209_SILENTSTEPSTICK
Connections:
- net at SW1.1, SW2.1, SW3.1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: now also U5.5 (VCC), U6.1 (VCC), U7.2 (VCC)
- net at SW7.2: now also R1.1, U1.11 (IO27)
- net at U1.33 (IO21): now also U5.2 (SDA), U7.3 (SDA)
- net at U1.36 (IO22): now also U5.3 (SCL), U7.4 (SCL)
- net at U1.38 (GND3): now also U5.4 (GND), U7.1 (GND)
- net at R4.1: now also SW2.2, U1.6 (IO35); no longer SW2.3
- net at SW5.2: now also R5.1, U1.9 (IO25)
- net at SW3.2: now also R7.1, U1.7 (IO32)
- net at SW4.2: now also R2.1, U1.8 (IO33)
- net at U1.32 (GND2): now also U6.4 (GND)
- net at U1.34 (RXD0): now also U6.2 (RX)
- net at U1.35 (TXD0): now also U6.3 (TX)
- net at U1.10 (IO26): now also R6.1, SW6.2; no longer SW6.4
- net at U1.5 (IO34): now also R3.1, SW1.2; no longer SW1.4
